Commit message: Pusher works.

File: urdf/common_properties.urdf.xacro (robot description, xacro)
@@ -40,4 +40,9 @@
     </material>
   </xacro:property>
+  <xacro:property name="material_neon_greeen">
+    <material name="neon_green">
+      <color rgba="0 1 0 1"/>
+    </material>
+  </xacro:property>
   <xacro:property name="material_blue">
     <material name="blue">

File: urdf/kobuki.urdf.xacro (robot description, xacro)
@@ -7,6 +7,6 @@
  -->
 <robot name="kobuki" xmlns:xacro="http://ros.org/wiki/xacro">
-  <xacro:include filename="$(find kobuki_description)/urdf/common_properties.urdf.xacro"/>
-  <xacro:include filename="$(find kobuki_description)/urdf/kobuki_gazebo.urdf.xacro"/>
+  <xacro:include filename="$(find learning_kobuki_description)/urdf/common_properties.urdf.xacro"/>
+  <xacro:include filename="$(find learning_kobuki_description)/urdf/kobuki_gazebo.urdf.xacro"/>
   <!-- Kobuki -->
   <xacro:macro name="kobuki">
@@ -30,5 +30,5 @@
         <geometry>
           <!-- new mesh -->
-          <mesh filename="package://kobuki_description/meshes/main_body.dae" />
+          <mesh filename="package://learning_kobuki_description/meshes/main_body.dae" />
         </geometry>
         <origin xyz="0.001 0 0.05199" rpy="0 0 0"/>
@@ -56,4 +56,36 @@
       </inertial>
     </link>
+    <joint name="pusher_joint" type="fixed">
+      <origin xyz="0 0 0.0102" rpy="0 0 0" />
+      <parent link="base_link"/>
+      <child link="pusher_link" />
+    </joint>
+    <link name="pusher_link">
+      <visual>
+        <geometry>
+          <!-- new mesh -->
+          <mesh filename="package://learning_kobuki_description/meshes/turtle_pusher.dae" />
+        </geometry>
+        <origin xyz="0.005 0 0.05199" rpy="0 0 0"/>
+        <material name="neon_green">
+          <color rgba="0 1 0 1"/>
+        </material>
+      </visual>
+      <collision>
+        <geometry>
+          <!-- Custom collision mesh -->
+          <mesh filename="package://learning_kobuki_description/meshes/turtle_pusher_collision.dae" />
+        </geometry>
+        <origin xyz="0.005 0 0.05199" rpy="0 0 0"/>
+      </collision>
+      <inertial>
+        <!-- COM experimentally determined -->
+        <origin xyz="0.015 0 0.05199"/>
+        <mass value="0.0"/> <!-- 2.4/2.6 kg for small/big battery pack -->
+        <inertia ixx="0.0" ixy="0.0" ixz="0.0"
+                 iyy="0.0" iyz="0.0"
+                 izz="0.0" />
+      </inertial>
+    </link>
     <joint name="wheel_left_joint" type="continuous">
       <parent link="base_link"/>
@@ -65,5 +97,5 @@
       <visual>
         <geometry>
-          <mesh filename="package://kobuki_description/meshes/wheel.dae"/>
+          <mesh filename="package://learning_kobuki_description/meshes/wheel.dae"/>
         </geometry>
         <origin xyz="0 0 0" rpy="0 0 0"/>
@@ -92,5 +124,5 @@
       <visual>
         <geometry>
-          <mesh filename="package://kobuki_description/meshes/wheel.dae"/>
+          <mesh filename="package://learning_kobuki_description/meshes/wheel.dae"/>
         </geometry>
         <origin xyz="0 0 0" rpy="0 0 0"/>

File: urdf/kobuki_gazebo.urdf.xacro (robot description, xacro)
@@ -9,4 +9,13 @@
 	    <minDepth>0.001</minDepth>
 	    <maxVel>1.0</maxVel>
+	  </gazebo>
+	  <gazebo reference="puser_link">
+	    <mu1>1.0</mu1>
+	    <mu2>1.0</mu2>
+	    <kp>1000000.0</kp>
+	    <kd>100.0</kd>
+	    <minDepth>0.001</minDepth>
+	    <maxVel>1.0</maxVel>
+        <material>Gazebo/Black</material>
 	  </gazebo>
 	  <gazebo reference="wheel_right_link">

File: urdf/kobuki_standalone.urdf.xacro (robot description, xacro)
@@ -6,5 +6,5 @@
        xmlns:xacro="http://ros.org/wiki/xacro">
   <!-- Defines the kobuki component tag. -->
-  <xacro:include filename="$(find kobuki_description)/urdf/kobuki.urdf.xacro" />
+  <xacro:include filename="$(find learning_kobuki_description)/urdf/kobuki.urdf.xacro" />
   <kobuki/>
 </robot>
