Commit message: Fixed Pusher

File: urdf/kobuki.urdf.xacro (robot description, xacro)
@@ -68,5 +68,5 @@
         </geometry>
         <origin xyz="0.005 0 0.05199" rpy="0 0 0"/>
-        <material name="neon_green">
+        <material name="blue">
           <color rgba="0 1 0 1"/>
         </material>
